File: kicad/button_mount/button_mount.sch (KiCad schematic (older format))
At the start: 8 parts, among them J1 SW Terminal, J2 LED Terminal, SW1 CROWN-SDB-201C

Commit message: Cancelled BBr1. Updated BBr2 to include 4x term blocks, smaller diam
Parts:
- J1: value SW Terminal -> OSTVN04A150; footprint TerminalBlocks_Phoenix:TerminalBlock_Phoenix_MPT-2.54mm_2pol -> button_mount:OSTVN04A150; symbol Connector:Screw_Terminal_01x02 -> Connector:Screw_Terminal_01x04
- J2: value LED Terminal -> OSTVN04A150; footprint TerminalBlocks_Phoenix:TerminalBlock_Phoenix_MPT-2.54mm_2pol -> button_mount:OSTVN04A150; symbol Connector:Screw_Terminal_01x02 -> Connector:Screw_Terminal_01x04
Connections:
- net COL_OUT: now also J1.3 (Pin_3), J1.4 (Pin_4); no longer J1.2 (Pin_2)
- net LED_A: now also J2.2 (Pin_2)
- net LED_K: now also J2.3 (Pin_3), J2.4 (Pin_4); no longer J2.2 (Pin_2)
- net ROW_IN: now also J1.2 (Pin_2)
Changed lines of the file:
@@
 LED_A
 $Comp
-L Connector:Screw_Terminal_01x02 J2
+L Connector:Screw_Terminal_01x04 J2
 U 1 1 60E548D2
-P 2650 2050
-F 0 "J2" H 2730 2042 50  0000 L CNN
-F 1 "LED Terminal" H 2730 1951 50  0000 L CNN
-F 2 "TerminalBlocks_Phoenix:TerminalBlock_Phoenix_MPT-2.54mm_2pol" H 2650 2050 50  0001 C CNN
-F 3 "~" H 2650 2050 50  0001 C CNN
-	1    2650 2050
+P 2750 2050
+F 0 "J2" H 2830 2042 50  0000 L CNN
+F 1 "OSTVN04A150" H 2830 1951 50  0000 L CNN
+F 2 "button_mount:OSTVN04A150" H 2750 2050 50  0001 C CNN
+F 3 "~" H 2750 2050 50  0001 C CNN
+	1    2750 2050
 	1    0    0    -1
 $EndComp
-Wire Wire Line
-	2450 2050 2150 2050
-Wire Wire Line
-	2150 2150 2450 2150
 Wire Wire Line
 	2150 2150 2150 2800
@@
 	1250 1500 2150 1500
 $Comp
-L Connector:Screw_Terminal_01x02 J1
+L Connector:Screw_Terminal_01x04 J1
 U 1 1 60E60A26
-P 2650 1050
-F 0 "J1" H 2730 1042 50  0000 L CNN
-F 1 "SW Terminal" H 2730 951 50  0000 L CNN
-F 2 "TerminalBlocks_Phoenix:TerminalBlock_Phoenix_MPT-2.54mm_2pol" H 2650 1050 50  0001 C CNN
-F 3 "~" H 2650 1050 50  0001 C CNN
-	1    2650 1050
+P 2750 1050
+F 0 "J1" H 2830 1042 50  0000 L CNN
+F 1 "OSTVN04A150" H 2830 951 50  0000 L CNN
+F 2 "button_mount:OSTVN04A150" H 2750 1050 50  0001 C CNN
+F 3 "~" H 2750 1050 50  0001 C CNN
+	1    2750 1050
 	1    0    0    -1
 $EndComp
-Text Notes 2250 2500 0    50   ~ 0
+Text Notes 2250 2600 0    50   ~ 0
 Driving options:\n- Connect as matrix\n- LED_A to VCC, LED_K to dedicated PWM pins\n
-Text Notes 2450 1300 2    50   ~ 0
+Text Notes 2350 1300 2    50   ~ 0
 Columns driven low, rows pulled high
-Wire Wire Line
-	1000 1150 2450 1150
 Text Label 1950 1150 0    50   ~ 0
 COL_OUT
-Wire Wire Line
-	1800 1050 2450 1050
 Text Label 1950 1050 0    50   ~ 0
 ROW_IN
@@
 	1    0    0    -1
 $EndComp
+Wire Wire Line
+	2150 2050 2450 2050
+Wire Wire Line
+	2450 2050 2450 1950
+Wire Wire Line
+	2450 1950 2550 1950
+Connection ~ 2450 2050
+Wire Wire Line
+	2450 2050 2550 2050
+Wire Wire Line
+	2150 2150 2450 2150
+Wire Wire Line
+	2450 2150 2450 2250
+Wire Wire Line
+	2450 2250 2550 2250
+Connection ~ 2450 2150
+Wire Wire Line
+	2450 2150 2550 2150
+Wire Wire Line
+	1800 1050 2450 1050
+Wire Wire Line
+	2450 1050 2450 950
+Wire Wire Line
+	2450 950  2550 950
+Connection ~ 2450 1050
+Wire Wire Line
+	2450 1050 2550 1050
+Wire Wire Line
+	1000 1150 2450 1150
+Wire Wire Line
+	2450 1150 2450 1250
+Wire Wire Line
+	2450 1250 2550 1250
+Connection ~ 2450 1150
+Wire Wire Line
+	2450 1150 2550 1150
 $EndSCHEMATC
